File: SOURCES/KiCAD/USBi_Programmer.kicad_pcb (KiCad board)
At the start: 2 copper layers, 40 x 47 mm, 34 parts, among them P1 CONN_02X10, P2 CONN_02X05, P3 CONN_01X02, P4 CONN_02X10, Q1 Q_NMOS_DGS, Q2 Q_NMOS_DGS, Q3 2N7002, Q4 2N7002

Commit message: Add files via upload
Parts:
- removed R10: 49R9, Resistors_SMD:R_0805_HandSoldering
- removed R11, R13, R16, R17, R18: 470R, Resistors_SMD:R_0805_HandSoldering
- removed R12, R15: 10k, Resistors_SMD:R_0805_HandSoldering
- removed R14: 1M, Resistors_SMD:R_0805_HandSoldering
- C2: value 100u -> 100uF
- D1, D2, D3, D4: footprint LEDs:LED-3MM -> LEDs:LED_D3.0mm
- P2: footprint Connectors_IDC:IDC-Header_2x05_Pitch2.54mm_Straight -> fdsp_connector:IDC_Header_Straight_10pins
- R1: value 49R9 -> 47R; footprint Resistors_THT:R_Axial_DIN0204_L3.6mm_D1.6mm_P7.62mm_Horizontal -> MyFootprints:Resistor_SMD+THTuniversal_0603to0805_RM7.5_HandSoldering_RevA_Date25Jun2010; moved to F.Cu
- R2, R3, R4, R5, R6, R7, R8, R9: footprint Resistors_THT:R_Axial_DIN0204_L3.6mm_D1.6mm_P7.62mm_Horizontal -> MyFootprints:Resistor_SMD+THTuniversal_0603to0805_RM7.5_HandSoldering_RevA_Date25Jun2010; moved to F.Cu
- moved R2 4.11 mm to (116.0, 160.8)
- moved R4 3.96 mm to (115.8, 157.4), turned to 0 degrees
- moved R3 3.67 mm to (115.8, 153.8), turned to 180 degrees
- moved R6 3.59 mm to (116.6, 146.3)
- moved R9 3.56 mm to (128.5, 146.4)
- moved R7 3.56 mm to (124.7, 146.4)
- moved R1 3.56 mm to (111.8, 146.4)
- moved R5 3.56 mm to (120.8, 146.4)
- moved R8 2.73 mm to (124.3, 167.0), turned to 180 degrees
- moved P2 0.51 mm to (115.1, 175.3), turned to 0 degrees
- moved C2 0.32 mm to (112.5, 165.5)
Connections:
- P1 pad 1: (no net) -> Net-(P1-Pad1)
- P1 pad 10: (no net) -> Net-(P1-Pad10)
- P1 pad 12: (no net) -> Net-(P1-Pad12)
- P1 pad 19: (no net) -> Net-(P1-Pad19)
- P1 pad 2: (no net) -> Net-(P1-Pad2)
- P1 pad 3: (no net) -> Net-(P1-Pad3)
- P1 pad 7: (no net) -> Net-(P1-Pad7)
- P1 pad 8: (no net) -> Net-(P1-Pad8)
- P4 pad 1: (no net) -> Net-(P4-Pad1)
- P4 pad 10: (no net) -> Net-(P4-Pad10)
- P4 pad 14: (no net) -> Net-(P4-Pad14)
- P4 pad 15: (no net) -> Net-(P4-Pad15)
- P4 pad 16: (no net) -> Net-(P4-Pad16)
- P4 pad 17: (no net) -> Net-(P4-Pad17)
- P4 pad 18: (no net) -> Net-(P4-Pad18)
- P4 pad 19: (no net) -> Net-(P4-Pad19)
- P4 pad 2: (no net) -> Net-(P4-Pad2)
- P4 pad 3: (no net) -> Net-(P4-Pad3)
- P4 pad 4: (no net) -> Net-(P4-Pad4)
- P4 pad 5: (no net) -> Net-(P4-Pad5)
- P4 pad 7: (no net) -> Net-(P4-Pad7)
- P4 pad 8: (no net) -> Net-(P4-Pad8)
- P4 pad 9: (no net) -> Net-(P4-Pad9)
Routing:
- net USB_PWR_ON: track 50.7 -> 64.8 mm
- net COUT: track 36.0 -> 25.5 mm, vias 1 -> 0
- net USB_CLK: track 27.4 -> 37.1 mm
- net SDA: track 33.8 -> 24.9 mm
- net Net-(P2-Pad3): track 35.9 -> 27.3 mm
- net Net-(P1-Pad5): track 19.5 -> 11.8 mm
- net +3V3: track 73.2 -> 66.2 mm
- net Net-(P2-Pad1): track 29.1 -> 23.7 mm
- net CCLK: track 37.9 -> 33.6 mm
- net SCL: track 35.5 -> 39.5 mm
- net LED_3: track 30.4 -> 27.0 mm
- net GND: track 2.33 -> 0.00 mm
- net LED_2: track 28.1 -> 25.9 mm
- net ~CLATCH1: track 23.4 -> 21.3 mm
- net CDATA: track 19.4 -> 17.5 mm
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Other:
- board text added: "BLU"
- board text added: "G S D"
- board text added: "RED"
- board text added: "TO TARGET DSP"
- board text added: "YEL"
- board text added: "freeUSBi v0.4"
- board text removed: "freeUSBi v0.3"

Commit message: Verion 0.5 update Release
Parts:
- C2: value 100uF -> 100u
- P2: footprint fdsp_connector:IDC_Header_Straight_10pins -> Connector_IDC:IDC-Header_2x05_P2.54mm_Horizontal
- R1: value 47R -> 49R9
- moved P2 10.4 mm to (125.0, 172.2), turned to 270 degrees
Connections:
- Q1 pad 2: USB_PWR_ON -> +3V3
- Q2 pad 2: USB_PWR_ON -> +3V3
- Q3 pad 1: USB_PWR_ON -> +3V3
- Q4 pad 1: USB_PWR_ON -> +3V3
- R3 pad 2: USB_PWR_ON -> +3V3
- R4 pad 1: USB_PWR_ON -> +3V3
- R8 pad 2: USB_PWR_ON -> +3V3
Routing:
- net +3V3: track 66.2 -> 159.9 mm, vias 0 -> 1
- net USB_PWR_ON: track 64.8 -> 0.00 mm
- net LED_1: track 22.0 -> 30.8 mm
- net SCL: track 39.5 -> 47.4 mm
- net +5VD: track 55.9 -> 63.3 mm
- net Net-(P2-Pad3): track 27.3 -> 22.0 mm, vias 0 -> 1
- net CDATA: track 17.5 -> 22.7 mm
- net ~CLATCH1: track 21.3 -> 25.6 mm
- net LED_3: track 27.0 -> 30.4 mm
- net COUT: track 25.5 -> 22.3 mm
- net CCLK: track 33.6 -> 30.5 mm
- net USB_CLK: track 37.1 -> 39.9 mm
- net SDA: track 24.9 -> 27.6 mm
- net GND: track 0.00 -> 2.75 mm
- net BRD_~RESET: track 15.1 -> 17.5 mm
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Other:
- board text added: "+"
- board text added: "A"
- board text added: "FreeUSBi v0.5"
- board text added: "K"
- board text removed: "freeUSBi v0.4"
