File: SOURCES/KiCAD/USBi_Programmer.sch (KiCad schematic (older format))
At the start: 32 parts, among them P1 CONN_02X10, P2 CONN_02X05, P3 CONN_01X02, P4 CONN_02X10, Q1 Q_NMOS_DGS, Q2 Q_NMOS_DGS, Q3 2N7002, Q4 2N7002

Commit message: Add files via upload
Parts:
- removed R10: 49R9, Resistors_SMD:R_0805_HandSoldering, symbol Device:R
- removed R11, R13, R16, R17, R18: 470R, Resistors_SMD:R_0805_HandSoldering, symbol Device:R
- removed R12, R15: 10k, Resistors_SMD:R_0805_HandSoldering, symbol Device:R
- removed R14: 1M, Resistors_SMD:R_0805_HandSoldering, symbol Device:R
- D1, D2, D3, D4: footprint LEDs:LED-3MM -> LEDs:LED_D3.0mm
- P2: footprint Connectors_IDC:IDC-Header_2x05_Pitch2.54mm_Straight -> fdsp_connector:IDC_Header_Straight_10pins
- R1, R2, R3, R4, R5, R6, R7, R8, R9: footprint Resistors_THT:R_Axial_DIN0204_L3.6mm_D1.6mm_P7.62mm_Horizontal -> MyFootprints:Resistor_SMD+THTuniversal_0603to0805_RM7.5_HandSoldering_RevA_Date25Jun2010
Other:
- note removed: "Note:\nParrallel connected parts are selectable choice.\nPlace your desired type one . (SMD or TH)\nNot needed both."

Commit message: Verion 0.5 update Release
Connections:
- net +3V3: now also Q1.2 (G), Q2.2 (G), Q3.1 (G), Q4.1 (G), R3.2, R4.1, R8.2
- net USB_PWR_ON: no longer Q1.2 (G), Q2.2 (G), Q3.1 (G), Q4.1 (G), R3.2, R4.1, R8.2
Other:
- note added: "JUMP to P1 pin20"
- note added: "Some FX2 board has an Non-bootable issue\nCause of I2C SDA voltage droped during boot."
Changed lines of the file:
@@
 EESchema Schematic File Version 4
-LIBS:USBi_Programmer-cache
-EELAYER 29 0
+EELAYER 30 0
 EELAYER END
 $Descr A4 11693 8268
 encoding utf-8
 Sheet 1 1
-Title "freeUSBi V0.4"
-Date "2019-05-11"
-Rev "0.4"
+Title "freeUSBi V0.5"
+Date "2025-05-03"
+Rev "0.5"
 Comp "www.freedsp.cc"
 Comment1 "www.creativecommons.org/licenses/by-sa/4.0/legalcode"
@@
 Text GLabel 5100 4950 0    51   Input ~ 0
 COUT
-Text GLabel 5100 4200 0    51   Input ~ 0
-USB_PWR_ON
 Text GLabel 8300 4400 2    51   Input ~ 0
 CDATA
@@
 P 5050 2850
 F 0 "#PWR08" H 5050 2700 50  0001 C CNN
-F 1 "+3.3V" V 5050 2990 50  0000 L TNN
+F 1 "+3.3V" V 5025 2950 50  0000 L TNN
 F 2 "" H 5050 2850 60  0000 C CNN
 F 3 "" H 5050 2850 60  0000 C CNN
@@
 	5100 3900 5500 3900
 Wire Wire Line
-	5100 4200 5500 4200
-Wire Wire Line
 	5100 4500 5500 4500
 Wire Wire Line
@@
 Wire Wire Line
 	6450 4200 6600 4200
+$Comp
+L power:+3.3V #PWR?
+U 1 1 68153F4C
+P 4925 4050
+F 0 "#PWR?" H 4925 3900 50  0001 C CNN
+F 1 "+3.3V" V 4900 4150 50  0000 L TNN
+F 2 "" H 4925 4050 60  0000 C CNN
+F 3 "" H 4925 4050 60  0000 C CNN
+	1    4925 4050
+	0    -1   -1   0
+$EndComp
+Wire Wire Line
+	4925 4050 5200 4050
+Wire Wire Line
+	5200 4050 5200 4200
+Wire Wire Line
+	5200 4200 5500 4200
+Wire Notes Line
+	4650 4000 4375 3750
+Wire Notes Line
+	4375 3750 4275 3750
+Text Notes 3150 3800 0    79   ~ 16
+JUMP to P1 pin20
+Text Notes 2625 3650 0    48   ~ 0
+Some FX2 board has an Non-bootable issue\nCause of I2C SDA voltage droped during boot.
 $EndSCHEMATC
