File: SOURCES/KiCAD/FreeUSBi.kicad_sch (KiCad schematic)
At the start: 23 parts, among them P1 CONN_02X10, P2 CONN_02X05, P3 CONN_01X02, P4 CONN_02X10, Q1 Q_NMOS_DGS, Q2 Q_NMOS_DGS, Q3 2N7002, Q4 2N7002

Commit message: Add files via upload
Parts:
- Q1, Q2: value Q_NMOS_DGS -> 2N7000
- R1: value 49R9 -> 47R
Changed lines of the file:
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@@
 			)
 		)
-		(property "Value" "49R9"
+		(property "Value" "47R"
 			(at 81.28 54.61 90)
 			(effects
@@
 			)
 		)
-		(property "Datasheet" ""
+		(property "Datasheet" "Any type of resistor is available"
 			(at 81.28 54.61 0)
 			(effects
@@
 					(size 0.762 0.762)
 				)
+				(hide yes)
 			)
 		)
@@
 			)
 		)
-		(property "Datasheet" ""
+		(property "Datasheet" "Any type of resistor is available"
 			(at 81.28 67.31 0)
 			(effects
@@
 					(size 0.762 0.762)
 				)
+				(hide yes)
 			)
 		)
@@
 			)
 		)
-		(property "Datasheet" ""
+		(property "Datasheet" "Any type of resistor is available"
 			(at 67.31 111.76 0)
 			(effects
@@
 					(size 0.762 0.762)
 				)
+				(hide yes)
 			)
 		)
@@
 			)
 		)
-		(property "Datasheet" ""
+		(property "Datasheet" "Any type of resistor is available"
 			(at 67.31 125.73 0)
 			(effects
@@
 					(size 0.762 0.762)
 				)
+				(hide yes)
 			)
 		)
@@
 			)
 		)
-		(property "Datasheet" ""
+		(property "Datasheet" "Any type of resistor is available"
 			(at 67.31 139.7 0)
 			(effects
@@
 					(size 0.762 0.762)
 				)
+				(hide yes)
 			)
 		)
@@
 		(dnp no)
 		(property "Reference" "Q1"
-			(at 157.48 100.33 90)
+			(at 156.464 99.822 90)
 			(effects
 				(font
@@
 			)
 		)
-		(property "Value" "Q_NMOS_DGS"
-			(at 167.005 102.87 90)
+		(property "Value" "2N7000"
+			(at 161.29 102.616 90)
 			(effects
 				(font
@@
 			)
 		)
-		(property "Datasheet" ""
+		(property "Datasheet" "Any type of resistor is available"
 			(at 139.7 102.87 0)
 			(effects
@@
 					(size 0.762 0.762)
 				)
+				(hide yes)
 			)
 		)
@@
 		(dnp no)
 		(property "Reference" "Q2"
-			(at 155.575 113.03 90)
+			(at 155.956 110.236 90)
 			(effects
 				(font
@@
 			)
 		)
-		(property "Value" "Q_NMOS_DGS"
-			(at 170.815 115.57 90)
+		(property "Value" "2N7000"
+			(at 160.782 111.252 90)
 			(effects
 				(font
@@
 			)
 		)
-		(property "Datasheet" ""
+		(property "Datasheet" "Any type of resistor is available"
 			(at 139.7 110.49 0)
 			(effects
@@
 					(size 0.762 0.762)
 				)
+				(hide yes)
 			)
 		)
@@
 			)
 		)
-		(property "Datasheet" ""
+		(property "Datasheet" "Any type of resistor is available"
 			(at 67.31 153.67 0)
 			(effects
@@
 					(size 0.762 0.762)
 				)
+				(hide yes)
 			)
 		)
@@
 			)
 		)
-		(property "Datasheet" ""
+		(property "Datasheet" "Any type of resistor is available"
 			(at 160.02 106.68 0)
 			(effects
@@
 					(size 0.762 0.762)
 				)
+				(hide yes)
 			)
 		)
@@
 			)
 		)
-		(property "Datasheet" "At least single Wire Connection Required(+5V)"
+		(property "Datasheet" "At least single Wire Connection Required(EZ-USB's +5V)"
 			(at 218.44 54.61 0)
 			(effects
@@
 					(size 1.524 1.524)
 				)
-			)
-		)
+				(hide yes)
+			)
+		)
